Commit message: First commit

File: husky_description/urdf/accessories/vlp16_mount.urdf.xacro (robot description, xacro)
@@ -1,4 +1,5 @@
 <?xml version="1.0"?>
 <robot xmlns:xacro="http://wiki.ros.org/xacro">
+  <xacro:property name="M_PI" value="3.1415926535897931" />
   <xacro:include filename="$(find velodyne_description)/urdf/VLP-16.urdf.xacro" />
   <xacro:macro name="vlp16_mount" params="prefix parent_link topic height:=0.12 *origin">
@@ -78,5 +79,5 @@
       <origin xyz="0 0 ${height}" rpy="0 0 0"/>
     </joint>
-    <xacro:VLP-16 parent="${prefix}vlp16_mount_plate" topic="${topic}">
+    <xacro:VLP-16 parent="${prefix}vlp16_mount_plate" topic="${topic}" gpu="true">
       <origin xyz="0 0 0" rpy="0 0 0" />
     </xacro:VLP-16>

File: husky_description/urdf/husky.urdf.xacro (robot description, xacro)
@@ -126,4 +126,13 @@
   <gazebo reference="imu_link">
   </gazebo>
+  <!-- GPS Link is the standard mounting position for the GPS-->
+  <link name="gps_link"/>
+  <joint name="gps_joint" type="fixed">
+    <origin xyz="$(optenv HUSKY_GPS_XYZ 0.0 0.0 0.5)" rpy="$(optenv HUSKY_GPS_RPY 0 0 0)" />
+    <parent link="base_link" />
+    <child link="gps_link" />
+  </joint>
+  <gazebo reference="gps_link">
+  </gazebo>
   <!-- Husky wheel macros -->
   <xacro:husky_wheel wheel_prefix="front_left">
@@ -227,11 +236,11 @@
     <plugin name="gps_controller" filename="libhector_gazebo_ros_gps.so">
       <robotNamespace>$(arg robot_namespace)</robotNamespace>
-      <updateRate>40</updateRate>
-      <bodyName>base_link</bodyName>
-      <frameId>base_link</frameId>
+      <updateRate>40.0</updateRate>
+      <bodyName>gps_link</bodyName>
+      <frameId>gps_link</frameId>
       <topicName>navsat/fix</topicName>
       <velocityTopicName>navsat/vel</velocityTopicName>
-      <referenceLatitude>49.9</referenceLatitude>
-      <referenceLongitude>8.9</referenceLongitude>
+      <referenceLatitude>48.711254</referenceLatitude>
+      <referenceLongitude>2.217765</referenceLongitude>
       <referenceHeading>0</referenceHeading>
       <referenceAltitude>0</referenceAltitude>

Commit message: Adding TEB Planner as an option for local planner but not using it because of its performances

File: husky_description/urdf/accessories/vlp16_mount.urdf.xacro (robot description, xacro)
@@ -1,7 +1,6 @@
 <?xml version="1.0"?>
 <robot xmlns:xacro="http://wiki.ros.org/xacro">
-  <xacro:property name="M_PI" value="3.1415926535897931" />
   <xacro:include filename="$(find velodyne_description)/urdf/VLP-16.urdf.xacro" />
-  <xacro:macro name="vlp16_mount" params="prefix parent_link topic height:=0.12 *origin">
+  <xacro:macro name="vlp16_mount" params="prefix parent_link topic height:=0.12 *origin gpu:=true">
     <!--
       The VLP16 is mounted to a pair of extrusion rods on top of the main sensor arch
@@ -57,11 +56,9 @@
       <origin xyz="0 -0.04 ${height/2}" rpy="0 0 0"/>
     </joint>
-<<<<<<< HEAD
     <xacro:VLP-16 parent="${prefix}vlp16_mount_base_link" topic="${topic}">
       <origin xyz="0 0 ${height}" rpy="0 0 0" />
-=======
     <xacro:VLP-16 parent="${prefix}vlp16_mount_plate" topic="${topic}" gpu="true">
+    <xacro:VLP-16 parent="${prefix}vlp16_mount_plate" topic="${topic}">
       <origin xyz="0 0 0" rpy="0 0 0" />
->>>>>>> c14491e... First commit
     </xacro:VLP-16>
   </xacro:macro>

Commit message: Adding TEB Planner as an option for local planner but not using it because of its performances

File: husky_description/urdf/accessories/vlp16_mount.urdf.xacro (robot description, xacro)
@@ -1,7 +1,6 @@
 <?xml version="1.0"?>
 <robot xmlns:xacro="http://wiki.ros.org/xacro">
-  <xacro:property name="M_PI" value="3.1415926535897931" />
   <xacro:include filename="$(find velodyne_description)/urdf/VLP-16.urdf.xacro" />
-  <xacro:macro name="vlp16_mount" params="prefix parent_link topic height:=0.12 *origin">
+  <xacro:macro name="vlp16_mount" params="prefix parent_link topic height:=0.12 *origin gpu:=true">
     <!--
       The VLP16 is mounted to a pair of extrusion rods on top of the main sensor arch
@@ -79,5 +78,5 @@
       <origin xyz="0 0 ${height}" rpy="0 0 0"/>
     </joint>
-    <xacro:VLP-16 parent="${prefix}vlp16_mount_plate" topic="${topic}" gpu="true">
+    <xacro:VLP-16 parent="${prefix}vlp16_mount_plate" topic="${topic}">
       <origin xyz="0 0 0" rpy="0 0 0" />
     </xacro:VLP-16>

Commit message: Adding ZED camera and RoboSense lidar descriptions

File: husky_description/urdf/accessories/vlp16_mount.urdf.xacro (robot description, xacro)
@@ -2,5 +2,5 @@
 <robot xmlns:xacro="http://wiki.ros.org/xacro">
   <xacro:include filename="$(find velodyne_description)/urdf/VLP-16.urdf.xacro" />
-  <xacro:macro name="vlp16_mount" params="prefix parent_link topic height:=0.12 *origin gpu:=true">
+  <xacro:macro name="vlp16_mount" params="prefix parent_link topic height:=0.12 *origin">
     <!--
       The VLP16 is mounted to a pair of extrusion rods on top of the main sensor arch
@@ -78,5 +78,5 @@
       <origin xyz="0 0 ${height}" rpy="0 0 0"/>
     </joint>
-    <xacro:VLP-16 parent="${prefix}vlp16_mount_plate" topic="${topic}">
+    <xacro:VLP-16 parent="${prefix}vlp16_mount_plate" topic="${topic}" gpu="true">
       <origin xyz="0 0 0" rpy="0 0 0" />
     </xacro:VLP-16>

File: husky_description/urdf/husky.urdf.xacro (robot description, xacro)
@@ -40,11 +40,19 @@
   <xacro:arg name="laser_ust10_rear_xyz"      default="$(optenv HUSKY_UST10_SECONDARY_XYZ -0.2206 0.0 0.00635)" />
   <xacro:arg name="laser_ust10_rear_rpy"      default="$(optenv HUSKY_UST10_SECONDARY_RPY 0 0 3.14159)" />
-  <xacro:arg name="laser_3d_enabled" default="$(optenv HUSKY_LASER_3D_ENABLED 1)" />
+  <xacro:arg name="laser_3d_enabled" default="$(optenv HUSKY_LASER_3D_ENABLED 0)" />
   <xacro:arg name="laser_3d_xyz" default="$(optenv HUSKY_LASER_3D_XYZ 0 0 0)" />
   <xacro:arg name="laser_3d_rpy" default="$(optenv HUSKY_LASER_3D_RPY 0 0 0)" />
-  <xacro:arg name="realsense_enabled" default="$(optenv HUSKY_REALSENSE_ENABLED 1)" />
+  <xacro:arg name="robosense_enabled" default="$(optenv HUSKY_ROBOSENSE_ENABLED 1)" />
+  <xacro:arg name="robosense_xyz" default="$(optenv HUSKY_ROBOSENSE_XYZ 0 0 0.08)" />
+  <xacro:arg name="robosense_rpy" default="$(optenv HUSKY_ROBOSENSE_RPY 0 0 0)" />
+  <xacro:arg name="realsense_enabled" default="$(optenv HUSKY_REALSENSE_ENABLED 0)" />
   <xacro:arg name="realsense_xyz" default="$(optenv HUSKY_REALSENSE_XYZ 0 0 0)" />
   <xacro:arg name="realsense_rpy" default="$(optenv HUSKY_REALSENSE_RPY 0 0 0)" />
   <xacro:arg name="realsense_mount" default="$(optenv HUSKY_REALSENSE_MOUNT_FRAME sensor_arch_mount_link)" />
+  <xacro:arg name="zed_enabled" default="$(optenv HUSKY_ZED_ENABLED 1)" />
+  <xacro:arg name="zed_xyz" default="$(optenv HUSKY_ZED_XYZ 0 0 0)" />
+  <xacro:arg name="zed_rpy" default="$(optenv HUSKY_ZED_RPY 0 0 0)" />
+  <xacro:arg name="zed_mount" default="$(optenv HUSKY_ZED_MOUNT_FRAME sensor_arch_mount_link)" />
+  <xacro:arg name="zed_model" default="$(optenv HUSKY_ZED_MODEL zed2)" />
   <xacro:property name="husky_front_bumper_extend" value="$(optenv HUSKY_FRONT_BUMPER_EXTEND 0)" />
   <xacro:property name="husky_rear_bumper_extend" value="$(optenv HUSKY_REAR_BUMPER_EXTEND 0)" />
@@ -59,8 +67,10 @@
   <xacro:include filename="$(find husky_description)/urdf/wheel.urdf.xacro" />
   <xacro:include filename="$(find husky_description)/urdf/accessories/intel_realsense.urdf.xacro"/>
+  <xacro:include filename="$(find zed_wrapper)/urdf/zed_macro.urdf.xacro" />
   <xacro:include filename="$(find husky_description)/urdf/accessories/hokuyo_ust10.urdf.xacro" />
   <xacro:include filename="$(find husky_description)/urdf/accessories/sick_lms1xx_mount.urdf.xacro"/>
   <xacro:include filename="$(find husky_description)/urdf/accessories/sensor_arch.urdf.xacro"/>
   <xacro:include filename="$(find husky_description)/urdf/accessories/vlp16_mount.urdf.xacro"/>
+  <xacro:include filename="$(find robosense_description)/urdf/RS-16.urdf.xacro"/>
   <xacro:property name="M_PI" value="3.14159"/>
   <!-- Base Size -->
@@ -189,6 +199,8 @@
   <xacro:property name="sensorbar_user_enabled"     value="$(arg sensor_arch)" />
   <xacro:property name="sensorbar_needed_realsense" value="$(arg realsense_enabled)" />
+  <xacro:property name="sensorbar_needed_zed"       value="$(arg zed_enabled)" />
   <xacro:property name="sensorbar_needed_lidar"     value="$(arg laser_3d_enabled)" />
-  <xacro:if value="${sensorbar_needed_realsense or sensorbar_user_enabled or sensorbar_needed_lidar}">
+  <xacro:property name="sensorbar_needed_robosense" value="$(arg robosense_enabled)" />
+  <xacro:if value="${sensorbar_needed_realsense or sensorbar_needed_zed or sensorbar_user_enabled or sensorbar_needed_lidar or sensorbar_needed_robosense}">
     <xacro:sensor_arch prefix="" parent="top_plate_link" size="$(arg sensor_arch_height)">
         <origin xyz="$(optenv HUSKY_SENSOR_ARCH_OFFSET 0 0 0)" rpy="$(optenv HUSKY_SENSOR_ARCH_RPY 0 0 0)"/>
@@ -205,4 +217,18 @@
     <xacro:intel_realsense_mount prefix="camera" topic="realsense" parent_link="realsense_mountpoint"/>
   </xacro:if>
+  <!-- add the zed camera to the sensor arch if needed -->
+  <xacro:unless value="$(arg realsense_enabled)">
+    <xacro:if value="$(arg zed_enabled)">
+      <link name="zed_mountpoint"/>
+      <joint name="zed_mountpoint_joint" type="fixed">
+        <origin xyz="$(arg zed_xyz)" rpy="$(arg zed_rpy)" />
+        <parent link="$(arg zed_mount)"/>
+        <child link="zed_mountpoint" />
+      </joint>
+      <xacro:zed_camera name="zed_node" model="$(arg zed_model)" parent="zed_mountpoint">
+        <origin xyz="$(arg zed_xyz)" rpy="$(arg zed_rpy)" />
+      </xacro:zed_camera>
+    </xacro:if>
+  </xacro:unless>
   <!--
     Add the 3d laser to the sensor arch if needed
@@ -213,4 +239,14 @@
     </xacro:vlp16_mount>
   </xacro:if>
+  <!--
+    Add the RoboSense 3D LiDAR to the sensor arch if needed
+  -->
+  <xacro:unless value="$(arg laser_3d_enabled)">
+    <xacro:if value="$(arg robosense_enabled)">
+      <xacro:RS-16 parent="sensor_arch_mount_link" name="robosense" topic="$(optenv HUSKY_ROBOSENSE_TOPIC rs_points)" hz="20" lasers="16" samples="900" collision_range="0.4" min_range="0.4" max_range="150.0" noise="0.008" gpu="true">
+        <origin xyz="$(arg robosense_xyz)" rpy="$(arg robosense_rpy)" />
+      </xacro:RS-16>
+    </xacro:if>
+  </xacro:unless>
   <gazebo>
     <plugin name="gazebo_ros_control" filename="libgazebo_ros_control.so">

Commit message: Adding ZED camera and RoboSense lidar descriptions

File: husky_description/urdf/accessories/vlp16_mount.urdf.xacro (robot description, xacro)
@@ -2,5 +2,5 @@
 <robot xmlns:xacro="http://wiki.ros.org/xacro">
   <xacro:include filename="$(find velodyne_description)/urdf/VLP-16.urdf.xacro" />
-  <xacro:macro name="vlp16_mount" params="prefix parent_link topic height:=0.12 *origin gpu:=true">
+  <xacro:macro name="vlp16_mount" params="prefix parent_link topic height:=0.12 *origin">
     <!--
       The VLP16 is mounted to a pair of extrusion rods on top of the main sensor arch
@@ -56,9 +56,6 @@
       <origin xyz="0 -0.04 ${height/2}" rpy="0 0 0"/>
     </joint>
-    <xacro:VLP-16 parent="${prefix}vlp16_mount_base_link" topic="${topic}">
+    <xacro:VLP-16 parent="${prefix}vlp16_mount_base_link" topic="${topic}" gpu="true">
       <origin xyz="0 0 ${height}" rpy="0 0 0" />
-    <xacro:VLP-16 parent="${prefix}vlp16_mount_plate" topic="${topic}" gpu="true">
-    <xacro:VLP-16 parent="${prefix}vlp16_mount_plate" topic="${topic}">
-      <origin xyz="0 0 0" rpy="0 0 0" />
     </xacro:VLP-16>
   </xacro:macro>

File: husky_description/urdf/husky.urdf.xacro (robot description, xacro)
@@ -40,11 +40,19 @@
   <xacro:arg name="laser_ust10_rear_xyz"      default="$(optenv HUSKY_UST10_SECONDARY_XYZ -0.2206 0.0 0.00635)" />
   <xacro:arg name="laser_ust10_rear_rpy"      default="$(optenv HUSKY_UST10_SECONDARY_RPY 0 0 3.14159)" />
-  <xacro:arg name="laser_3d_enabled" default="$(optenv HUSKY_LASER_3D_ENABLED 1)" />
+  <xacro:arg name="laser_3d_enabled" default="$(optenv HUSKY_LASER_3D_ENABLED 0)" />
   <xacro:arg name="laser_3d_xyz" default="$(optenv HUSKY_LASER_3D_XYZ 0 0 0)" />
   <xacro:arg name="laser_3d_rpy" default="$(optenv HUSKY_LASER_3D_RPY 0 0 0)" />
-  <xacro:arg name="realsense_enabled" default="$(optenv HUSKY_REALSENSE_ENABLED 1)" />
+  <xacro:arg name="robosense_enabled" default="$(optenv HUSKY_ROBOSENSE_ENABLED 1)" />
+  <xacro:arg name="robosense_xyz" default="$(optenv HUSKY_ROBOSENSE_XYZ 0 0 0.08)" />
+  <xacro:arg name="robosense_rpy" default="$(optenv HUSKY_ROBOSENSE_RPY 0 0 0)" />
+  <xacro:arg name="realsense_enabled" default="$(optenv HUSKY_REALSENSE_ENABLED 0)" />
   <xacro:arg name="realsense_xyz" default="$(optenv HUSKY_REALSENSE_XYZ 0 0 0)" />
   <xacro:arg name="realsense_rpy" default="$(optenv HUSKY_REALSENSE_RPY 0 0 0)" />
   <xacro:arg name="realsense_mount" default="$(optenv HUSKY_REALSENSE_MOUNT_FRAME sensor_arch_mount_link)" />
+  <xacro:arg name="zed_enabled" default="$(optenv HUSKY_ZED_ENABLED 1)" />
+  <xacro:arg name="zed_xyz" default="$(optenv HUSKY_ZED_XYZ 0 0 0)" />
+  <xacro:arg name="zed_rpy" default="$(optenv HUSKY_ZED_RPY 0 0 0)" />
+  <xacro:arg name="zed_mount" default="$(optenv HUSKY_ZED_MOUNT_FRAME sensor_arch_mount_link)" />
+  <xacro:arg name="zed_model" default="$(optenv HUSKY_ZED_MODEL zed2)" />
   <xacro:property name="husky_front_bumper_extend" value="$(optenv HUSKY_FRONT_BUMPER_EXTEND 0)" />
   <xacro:property name="husky_rear_bumper_extend" value="$(optenv HUSKY_REAR_BUMPER_EXTEND 0)" />
@@ -59,8 +67,11 @@
   <xacro:include filename="$(find husky_description)/urdf/wheel.urdf.xacro" />
   <xacro:include filename="$(find husky_description)/urdf/accessories/intel_realsense.urdf.xacro"/>
+  <xacro:include filename="$(find zed_wrapper)/urdf/zed_macro.urdf.xacro" />
+  <xacro:include filename="$(find husky_description)/urdf/accessories/hokuyo_ust10.urdf.xacro" />
   <xacro:include filename="$(find husky_description)/urdf/accessories/sick_lms1xx_mount.urdf.xacro"/>
   <xacro:include filename="$(find husky_description)/urdf/accessories/sensor_arch.urdf.xacro"/>
   <xacro:include filename="$(find husky_description)/urdf/accessories/hokuyo_ust10.urdf.xacro"/>
   <xacro:include filename="$(find husky_description)/urdf/accessories/vlp16_mount.urdf.xacro"/>
+  <xacro:include filename="$(find robosense_description)/urdf/RS-16.urdf.xacro"/>
   <xacro:property name="M_PI" value="3.14159"/>
   <!-- Base Size -->
@@ -189,6 +200,8 @@
   <xacro:property name="sensorbar_user_enabled"     value="$(arg sensor_arch)" />
   <xacro:property name="sensorbar_needed_realsense" value="$(arg realsense_enabled)" />
+  <xacro:property name="sensorbar_needed_zed"       value="$(arg zed_enabled)" />
   <xacro:property name="sensorbar_needed_lidar"     value="$(arg laser_3d_enabled)" />
-  <xacro:if value="${sensorbar_needed_realsense or sensorbar_user_enabled or sensorbar_needed_lidar}">
+  <xacro:property name="sensorbar_needed_robosense" value="$(arg robosense_enabled)" />
+  <xacro:if value="${sensorbar_needed_realsense or sensorbar_needed_zed or sensorbar_user_enabled or sensorbar_needed_lidar or sensorbar_needed_robosense}">
     <xacro:sensor_arch prefix="" parent="top_plate_link" size="$(arg sensor_arch_height)">
         <origin xyz="$(optenv HUSKY_SENSOR_ARCH_OFFSET 0 0 0)" rpy="$(optenv HUSKY_SENSOR_ARCH_RPY 0 0 0)"/>
@@ -205,4 +218,18 @@
     <xacro:intel_realsense_mount prefix="camera" topic="realsense" parent_link="realsense_mountpoint"/>
   </xacro:if>
+  <!-- add the zed camera to the sensor arch if needed -->
+  <xacro:unless value="$(arg realsense_enabled)">
+    <xacro:if value="$(arg zed_enabled)">
+      <link name="zed_mountpoint"/>
+      <joint name="zed_mountpoint_joint" type="fixed">
+        <origin xyz="$(arg zed_xyz)" rpy="$(arg zed_rpy)" />
+        <parent link="$(arg zed_mount)"/>
+        <child link="zed_mountpoint" />
+      </joint>
+      <xacro:zed_camera name="zed_node" model="$(arg zed_model)" parent="zed_mountpoint">
+        <origin xyz="$(arg zed_xyz)" rpy="$(arg zed_rpy)" />
+      </xacro:zed_camera>
+    </xacro:if>
+  </xacro:unless>
   <!--
     Add the 3d laser to the sensor arch if needed
@@ -213,4 +240,14 @@
     </xacro:vlp16_mount>
   </xacro:if>
+  <!--
+    Add the RoboSense 3D LiDAR to the sensor arch if needed
+  -->
+  <xacro:unless value="$(arg laser_3d_enabled)">
+    <xacro:if value="$(arg robosense_enabled)">
+      <xacro:RS-16 parent="sensor_arch_mount_link" name="robosense" topic="$(optenv HUSKY_ROBOSENSE_TOPIC rs_points)" hz="20" lasers="16" samples="900" collision_range="0.4" min_range="0.4" max_range="150.0" noise="0.008" gpu="true">
+        <origin xyz="$(arg robosense_xyz)" rpy="$(arg robosense_rpy)" />
+      </xacro:RS-16>
+    </xacro:if>
+  </xacro:unless>
   <gazebo>
     <plugin name="gazebo_ros_control" filename="libgazebo_ros_control.so">
