Commit message: Tweaking Husky config and parameters

File: husky_description/urdf/accessories/RS-16.urdf.xacro (robot description, xacro)
@@ -2,5 +2,5 @@
 <robot xmlns:xacro="http://www.ros.org/wiki/xacro" name="RS-16">
   <xacro:property name="M_PI" value="3.1415926535897931" />
-  <xacro:macro name="RS-16" params="*origin parent:=base_link name:=robosense topic:=/robosense_points hz:=20 lasers:=16 samples:=900 collision_range:=0.4 min_range:=0.4 max_range:=150.0 noise:=0.008 min_angle:=-${M_PI} max_angle:=${M_PI} gpu:=false">
+  <xacro:macro name="RS-16" params="*origin parent:=base_link name:=rslidar topic:=/rs_points hz:=20 lasers:=16 samples:=900 collision_range:=0.4 min_range:=0.4 max_range:=150.0 noise:=0.008 min_angle:=-${M_PI} max_angle:=${M_PI} gpu:=false">
     <joint name="${name}_base_mount_joint" type="fixed">
       <xacro:insert_block name="origin" />

File: husky_description/urdf/husky.urdf.xacro (robot description, xacro)
@@ -44,5 +44,5 @@
   <xacro:arg name="laser_3d_rpy" default="$(optenv HUSKY_LASER_3D_RPY 0 0 0)" />
   <xacro:arg name="robosense_enabled" default="$(optenv HUSKY_ROBOSENSE_ENABLED 1)" />
-  <xacro:arg name="robosense_xyz" default="$(optenv HUSKY_ROBOSENSE_XYZ -0.02 0 0.006)" />
+  <xacro:arg name="robosense_xyz" default="$(optenv HUSKY_ROBOSENSE_XYZ 0 0 0.044)" />
   <xacro:arg name="robosense_rpy" default="$(optenv HUSKY_ROBOSENSE_RPY 0 0 0)" />
   <xacro:arg name="realsense_enabled" default="$(optenv HUSKY_REALSENSE_ENABLED 0)" />
@@ -51,6 +51,6 @@
   <xacro:arg name="realsense_mount" default="$(optenv HUSKY_REALSENSE_MOUNT_FRAME sensor_arch_mount_link)" />
   <xacro:arg name="zed_enabled" default="$(optenv HUSKY_ZED_ENABLED 1)" />
-  <xacro:arg name="zed_xyz" default="$(optenv HUSKY_ZED_XYZ 0 0 -0.025)" />
-  <xacro:arg name="zed_rpy" default="$(optenv HUSKY_ZED_RPY 0 3.141593 0)" />
+  <xacro:arg name="zed_xyz" default="$(optenv HUSKY_ZED_XYZ 0 0 -0.265)" />
+  <xacro:arg name="zed_rpy" default="$(optenv HUSKY_ZED_RPY 0 0.05 0)" />
   <xacro:arg name="zed_mount" default="$(optenv HUSKY_ZED_MOUNT_FRAME sensor_arch_mount_link)" />
   <xacro:arg name="zed_model" default="$(optenv HUSKY_ZED_MODEL zed2)" />
@@ -133,5 +133,5 @@
   <link name="imu_link"/>
   <joint name="imu_joint" type="fixed">
-    <origin xyz="$(optenv HUSKY_IMU_XYZ 0 0 -0.54)" rpy="$(optenv HUSKY_IMU_RPY 0 -1.5708 3.1416)" />
+    <origin xyz="$(optenv HUSKY_IMU_XYZ 0 0 -0.3)" rpy="$(optenv HUSKY_IMU_RPY 3.141593 0 0)" />
     <parent link="sensor_arch_mount_link" />
     <child link="imu_link" />
@@ -142,5 +142,5 @@
   <link name="gps_link"/>
   <joint name="gps_joint" type="fixed">
-    <origin xyz="$(optenv HUSKY_GPS_XYZ -0.1 0 -0.27)" rpy="$(optenv HUSKY_GPS_RPY 0 0 0)" />
+    <origin xyz="$(optenv HUSKY_GPS_XYZ 0 0.22 0)" rpy="$(optenv HUSKY_GPS_RPY 0 0 0)" />
     <parent link="sensor_arch_mount_link" />
     <child link="gps_link" />
@@ -229,6 +229,6 @@
         <child link="zed_mountpoint" />
       </joint>
-      <xacro:zed_camera name="zed_node" model="$(arg zed_model)" parent="zed_mountpoint">
-        <origin xyz="0 0 0" rpy="0 -0.05 0" />
+      <xacro:zed_camera name="zed" model="$(arg zed_model)" parent="zed_mountpoint">
+        <origin xyz="0 0 0" rpy="0 0 0" />
       </xacro:zed_camera>
     </xacro:if>
@@ -247,11 +247,11 @@
   <xacro:unless value="$(arg laser_3d_enabled)">
     <xacro:if value="$(arg robosense_enabled)">
-	  <joint name="robosense_joint" type="fixed" >
-	    <parent link="sensor_arch_mount_link" />
-		<child link="robosense_mountpoint" />
-		<origin xyz="$(arg robosense_xyz)" rpy="$(arg robosense_rpy)" />
-	  </joint>
-	  <link name="robosense_mountpoint"/>
-      <xacro:RS-16 parent="robosense_mountpoint" name="robosense" topic="$(optenv HUSKY_ROBOSENSE_TOPIC rslidar_points)" hz="20" lasers="16" samples="900" collision_range="0.4" min_range="0.4" max_range="150.0" noise="0.008" gpu="true">
+      <joint name="robosense_joint" type="fixed" >
+        <parent link="sensor_arch_mount_link" />
+        <child link="robosense_mountpoint" />
+        <origin xyz="$(arg robosense_xyz)" rpy="$(arg robosense_rpy)" />
+      </joint>
+      <link name="robosense_mountpoint"/>
+      <xacro:RS-16 parent="robosense_mountpoint" name="rslidar" topic="$(optenv HUSKY_ROBOSENSE_TOPIC rslidar_points)" hz="20" lasers="16" samples="900" collision_range="0.4" min_range="0.4" max_range="150.0" noise="0.008" gpu="true">
         <origin xyz="0 0 0.008" rpy="0 0 0" />
       </xacro:RS-16>
@@ -282,5 +282,5 @@
       <robotNamespace>$(arg robot_namespace)</robotNamespace>
       <updateRate>40.0</updateRate>
-      <bodyName>gps_link</bodyName>
+      <bodyName>base_link</bodyName>
       <frameId>gps_link</frameId>
       <topicName>navsat/fix</topicName>

Commit message: Setting new architecture description, modifying localization configuration because of SBG IMU drivers (/imu/data message) has been changed to point toward 0 when facing East, actually adding web_video_server and possibility to record rosbag on external disk

File: husky_description/urdf/accessories/RS-16.urdf.xacro (robot description, xacro)
@@ -23,5 +23,5 @@
       </visual>
       <collision>
-        <origin rpy="0 0 0" xyz="0 0 0"/>
+        <origin rpy="0 0 0" xyz="0 0 0.0335"/>
         <geometry>
           <cylinder radius="0.0535" length="0.0817"/>

File: husky_description/urdf/accessories/sensor_arch.urdf.xacro (robot description, xacro)
@@ -1,4 +1,4 @@
 <?xml version="1.0"?>
-<robot xmlns:xacro="http://ros.org/wiki/xacro" name="510_mm_sensor_arch">
+<robot xmlns:xacro="http://ros.org/wiki/xacro" name="sensor_arch">
     <xacro:macro name="sensor_arch" params="prefix parent size:=510 *origin">
         <link name="${prefix}sensor_arch_base_link" />

File: husky_description/urdf/husky.urdf.xacro (robot description, xacro)
@@ -45,5 +45,5 @@
   <xacro:arg name="laser_3d_rpy" default="$(optenv HUSKY_LASER_3D_RPY 0 0 0)" />
   <xacro:arg name="robosense_enabled" default="$(optenv HUSKY_ROBOSENSE_ENABLED 1)" />
-  <xacro:arg name="robosense_xyz" default="$(optenv HUSKY_ROBOSENSE_XYZ 0.017 0 -0.135)" />
+  <xacro:arg name="robosense_xyz" default="$(optenv HUSKY_ROBOSENSE_XYZ 0 0 -0.33)" />
   <xacro:arg name="robosense_rpy" default="$(optenv HUSKY_ROBOSENSE_RPY 0 0 0)" />
   <xacro:arg name="realsense_enabled" default="$(optenv HUSKY_REALSENSE_ENABLED 0)" />
@@ -52,12 +52,12 @@
   <xacro:arg name="realsense_mount" default="$(optenv HUSKY_REALSENSE_MOUNT_FRAME sensor_arch_mount_link)" />
   <xacro:arg name="zed_enabled" default="$(optenv HUSKY_ZED_ENABLED 1)" />
-  <xacro:arg name="zed_xyz" default="$(optenv HUSKY_ZED_XYZ 0 0 -0.265)" />
-  <xacro:arg name="zed_rpy" default="$(optenv HUSKY_ZED_RPY 0 0.05 0)" />
+  <xacro:arg name="zed_xyz" default="$(optenv HUSKY_ZED_XYZ 0 0 -0.18)" />
+  <xacro:arg name="zed_rpy" default="$(optenv HUSKY_ZED_RPY 0 0.197 0)" />
   <xacro:arg name="zed_mount" default="$(optenv HUSKY_ZED_MOUNT_FRAME sensor_arch_mount_link)" />
   <xacro:arg name="zed_model" default="$(optenv HUSKY_ZED_MODEL zed2)" />
   <xacro:property name="husky_front_bumper_extend" value="$(optenv HUSKY_FRONT_BUMPER_EXTEND 0)" />
   <xacro:property name="husky_rear_bumper_extend" value="$(optenv HUSKY_REAR_BUMPER_EXTEND 0)" />
-  <!-- Height of the sensor arch in mm.  Must be either 540 or 510 or 300 -->
-  <xacro:arg name="sensor_arch_height"  default="$(optenv HUSKY_SENSOR_ARCH_HEIGHT 540)" />
+  <!-- Height of the sensor arch in mm.  Must be either 560 or 540 or 510 or 300 -->
+  <xacro:arg name="sensor_arch_height"  default="$(optenv HUSKY_SENSOR_ARCH_HEIGHT 560)" />
   <xacro:arg name="sensor_arch"         default="$(optenv HUSKY_SENSOR_ARCH 0)" />
   <xacro:arg name="sensor_arch_xyz"  default="$(optenv HUSKY_SENSOR_ARCH_OFFSET 0.01 0 0)" />
@@ -76,5 +76,4 @@
   <xacro:include filename="$(find husky_description)/urdf/accessories/sick_lms1xx_mount.urdf.xacro"/>
   <xacro:include filename="$(find husky_description)/urdf/accessories/sensor_arch.urdf.xacro"/>
-  <xacro:include filename="$(find husky_description)/urdf/accessories/hokuyo_ust10.urdf.xacro"/>
   <xacro:include filename="$(find husky_description)/urdf/accessories/vlp16_mount.urdf.xacro"/>
   <xacro:if value="$(arg robosense_enabled)">
@@ -139,5 +138,5 @@
   <xacro:if value="$(arg husky_sim)">
     <joint name="imu_joint" type="fixed">
-      <origin xyz="$(optenv HUSKY_IMU_XYZ 0 0 -0.3)" rpy="$(optenv HUSKY_IMU_RPY 0 -1.5708 3.1416)" />
+      <origin xyz="$(optenv HUSKY_IMU_XYZ 0 0 -0.38)" rpy="$(optenv HUSKY_IMU_RPY 0 0 0)" />
       <parent link="sensor_arch_mount_link" />
       <child link="imu_link" />
@@ -146,5 +145,5 @@
   <xacro:unless value="$(arg husky_sim)">
     <joint name="imu_joint" type="fixed">
-      <origin xyz="$(optenv HUSKY_IMU_XYZ 0 0 -0.3)" rpy="$(optenv HUSKY_IMU_RPY 0 0 0)" />
+      <origin xyz="$(optenv HUSKY_IMU_XYZ 0 0 -0.38)" rpy="$(optenv HUSKY_IMU_RPY 0 0 0)" />
       <parent link="sensor_arch_mount_link" />
       <child link="imu_link" />
@@ -153,8 +152,21 @@
   <gazebo reference="imu_link">
   </gazebo>
+  <!-- GNSS Links is the standard mounting position for the SBG IMU dual GNSS-->
+  <link name="left_imu_gnss_link"/>
+  <joint name="left_imu_gnss_joint" type="fixed">
+    <origin xyz="0 0.25 0.01" rpy="0 0 0" />
+    <parent link="sensor_arch_mount_link" />
+    <child link="left_imu_gnss_link" />
+  </joint>
+  <link name="right_imu_gnss_link"/>
+  <joint name="right_imu_gnss_joint" type="fixed">
+    <origin xyz="0 -0.25 0.01" rpy="0 0 0" />
+    <parent link="sensor_arch_mount_link" />
+    <child link="right_imu_gnss_link" />
+  </joint>
   <!-- GPS Link is the standard mounting position for the GPS-->
   <link name="gps_link"/>
   <joint name="gps_joint" type="fixed">
-    <origin xyz="$(optenv HUSKY_GPS_XYZ 0 0.22 0)" rpy="$(optenv HUSKY_GPS_RPY 0 0 0)" />
+    <origin xyz="$(optenv HUSKY_GPS_XYZ 0 0.2 0.01)" rpy="$(optenv HUSKY_GPS_RPY 0 0 0)" />
     <parent link="sensor_arch_mount_link" />
     <child link="gps_link" />
