Commit message: Adapting URDF/description to the actual shape

File: husky_description/urdf/husky.urdf.xacro (robot description, xacro)
@@ -44,5 +44,5 @@
   <xacro:arg name="laser_3d_rpy" default="$(optenv HUSKY_LASER_3D_RPY 0 0 0)" />
   <xacro:arg name="robosense_enabled" default="$(optenv HUSKY_ROBOSENSE_ENABLED 1)" />
-  <xacro:arg name="robosense_xyz" default="$(optenv HUSKY_ROBOSENSE_XYZ 0 0 0.08)" />
+  <xacro:arg name="robosense_xyz" default="$(optenv HUSKY_ROBOSENSE_XYZ -0.02 0 0.006)" />
   <xacro:arg name="robosense_rpy" default="$(optenv HUSKY_ROBOSENSE_RPY 0 0 0)" />
   <xacro:arg name="realsense_enabled" default="$(optenv HUSKY_REALSENSE_ENABLED 0)" />
@@ -51,13 +51,15 @@
   <xacro:arg name="realsense_mount" default="$(optenv HUSKY_REALSENSE_MOUNT_FRAME sensor_arch_mount_link)" />
   <xacro:arg name="zed_enabled" default="$(optenv HUSKY_ZED_ENABLED 1)" />
-  <xacro:arg name="zed_xyz" default="$(optenv HUSKY_ZED_XYZ 0 0 0)" />
-  <xacro:arg name="zed_rpy" default="$(optenv HUSKY_ZED_RPY 0 0 0)" />
+  <xacro:arg name="zed_xyz" default="$(optenv HUSKY_ZED_XYZ 0 0 -0.025)" />
+  <xacro:arg name="zed_rpy" default="$(optenv HUSKY_ZED_RPY 0 3.141593 0)" />
   <xacro:arg name="zed_mount" default="$(optenv HUSKY_ZED_MOUNT_FRAME sensor_arch_mount_link)" />
   <xacro:arg name="zed_model" default="$(optenv HUSKY_ZED_MODEL zed2)" />
   <xacro:property name="husky_front_bumper_extend" value="$(optenv HUSKY_FRONT_BUMPER_EXTEND 0)" />
   <xacro:property name="husky_rear_bumper_extend" value="$(optenv HUSKY_REAR_BUMPER_EXTEND 0)" />
-  <!-- Height of the sensor arch in mm.  Must be either 510 or 300 -->
-  <xacro:arg name="sensor_arch_height"  default="$(optenv HUSKY_SENSOR_ARCH_HEIGHT 510)" />
+  <!-- Height of the sensor arch in mm.  Must be either 540 or 510 or 300 -->
+  <xacro:arg name="sensor_arch_height"  default="$(optenv HUSKY_SENSOR_ARCH_HEIGHT 540)" />
   <xacro:arg name="sensor_arch"         default="$(optenv HUSKY_SENSOR_ARCH 0)" />
+  <xacro:arg name="sensor_arch_xyz"  default="$(optenv HUSKY_SENSOR_ARCH_OFFSET 0.01 0 0)" />
+  <xacro:arg name="sensor_arch_rpy"     default="$(optenv HUSKY_SENSOR_ARCH_RPY 0 0 0)" />
   <xacro:arg name="robot_namespace" default="$(optenv ROBOT_NAMESPACE /)" />
   <xacro:arg name="urdf_extras" default="$(optenv HUSKY_URDF_EXTRAS empty.urdf)" />
@@ -130,6 +132,6 @@
   <link name="imu_link"/>
   <joint name="imu_joint" type="fixed">
-    <origin xyz="$(optenv HUSKY_IMU_XYZ 0.19 0 0.149)" rpy="$(optenv HUSKY_IMU_RPY 0 -1.5708 3.1416)" />
-    <parent link="base_link" />
+    <origin xyz="$(optenv HUSKY_IMU_XYZ 0 0 -0.54)" rpy="$(optenv HUSKY_IMU_RPY 0 -1.5708 3.1416)" />
+    <parent link="sensor_arch_mount_link" />
     <child link="imu_link" />
   </joint>
@@ -139,6 +141,6 @@
   <link name="gps_link"/>
   <joint name="gps_joint" type="fixed">
-    <origin xyz="$(optenv HUSKY_GPS_XYZ 0.0 0.0 0.5)" rpy="$(optenv HUSKY_GPS_RPY 0 0 0)" />
-    <parent link="base_link" />
+    <origin xyz="$(optenv HUSKY_GPS_XYZ -0.1 0 -0.27)" rpy="$(optenv HUSKY_GPS_RPY 0 0 0)" />
+    <parent link="sensor_arch_mount_link" />
     <child link="gps_link" />
   </joint>
@@ -204,6 +206,6 @@
   <xacro:if value="${sensorbar_needed_realsense or sensorbar_needed_zed or sensorbar_user_enabled or sensorbar_needed_lidar or sensorbar_needed_robosense}">
     <xacro:sensor_arch prefix="" parent="top_plate_link" size="$(arg sensor_arch_height)">
-        <origin xyz="$(optenv HUSKY_SENSOR_ARCH_OFFSET 0 0 0)" rpy="$(optenv HUSKY_SENSOR_ARCH_RPY 0 0 0)"/>
-      </xacro:sensor_arch>
+    	<origin xyz="$(arg sensor_arch_xyz)" rpy="$(arg sensor_arch_rpy)"/>
+    </xacro:sensor_arch>
   </xacro:if>
   <!-- add the intel realsense to the sensor arch if needed -->
@@ -227,5 +229,5 @@
       </joint>
       <xacro:zed_camera name="zed_node" model="$(arg zed_model)" parent="zed_mountpoint">
-        <origin xyz="$(arg zed_xyz)" rpy="$(arg zed_rpy)" />
+        <origin xyz="0 0 0" rpy="0 -0.05 0" />
       </xacro:zed_camera>
     </xacro:if>
@@ -244,6 +246,12 @@
   <xacro:unless value="$(arg laser_3d_enabled)">
     <xacro:if value="$(arg robosense_enabled)">
-      <xacro:RS-16 parent="sensor_arch_mount_link" name="robosense" topic="$(optenv HUSKY_ROBOSENSE_TOPIC rs_points)" hz="20" lasers="16" samples="900" collision_range="0.4" min_range="0.4" max_range="150.0" noise="0.008" gpu="true">
-        <origin xyz="$(arg robosense_xyz)" rpy="$(arg robosense_rpy)" />
+	  <joint name="robosense_joint" type="fixed" >
+	    <parent link="sensor_arch_mount_link" />
+		<child link="robosense_mountpoint" />
+		<origin xyz="$(arg robosense_xyz)" rpy="$(arg robosense_rpy)" />
+	  </joint>
+	  <link name="robosense_mountpoint"/>
+      <xacro:RS-16 parent="robosense_mountpoint" name="robosense" topic="$(optenv HUSKY_ROBOSENSE_TOPIC rslidar_points)" hz="20" lasers="16" samples="900" collision_range="0.4" min_range="0.4" max_range="150.0" noise="0.008" gpu="true">
+        <origin xyz="0 0 0.008" rpy="0 0 0" />
       </xacro:RS-16>
     </xacro:if>

Commit message: Adapting URDF/description to the actual shape

File: husky_description/urdf/husky.urdf.xacro (robot description, xacro)
@@ -44,5 +44,5 @@
   <xacro:arg name="laser_3d_rpy" default="$(optenv HUSKY_LASER_3D_RPY 0 0 0)" />
   <xacro:arg name="robosense_enabled" default="$(optenv HUSKY_ROBOSENSE_ENABLED 1)" />
-  <xacro:arg name="robosense_xyz" default="$(optenv HUSKY_ROBOSENSE_XYZ 0 0 0.08)" />
+  <xacro:arg name="robosense_xyz" default="$(optenv HUSKY_ROBOSENSE_XYZ -0.02 0 0.006)" />
   <xacro:arg name="robosense_rpy" default="$(optenv HUSKY_ROBOSENSE_RPY 0 0 0)" />
   <xacro:arg name="realsense_enabled" default="$(optenv HUSKY_REALSENSE_ENABLED 0)" />
@@ -51,13 +51,15 @@
   <xacro:arg name="realsense_mount" default="$(optenv HUSKY_REALSENSE_MOUNT_FRAME sensor_arch_mount_link)" />
   <xacro:arg name="zed_enabled" default="$(optenv HUSKY_ZED_ENABLED 1)" />
-  <xacro:arg name="zed_xyz" default="$(optenv HUSKY_ZED_XYZ 0 0 0)" />
-  <xacro:arg name="zed_rpy" default="$(optenv HUSKY_ZED_RPY 0 0 0)" />
+  <xacro:arg name="zed_xyz" default="$(optenv HUSKY_ZED_XYZ 0 0 -0.025)" />
+  <xacro:arg name="zed_rpy" default="$(optenv HUSKY_ZED_RPY 0 3.141593 0)" />
   <xacro:arg name="zed_mount" default="$(optenv HUSKY_ZED_MOUNT_FRAME sensor_arch_mount_link)" />
   <xacro:arg name="zed_model" default="$(optenv HUSKY_ZED_MODEL zed2)" />
   <xacro:property name="husky_front_bumper_extend" value="$(optenv HUSKY_FRONT_BUMPER_EXTEND 0)" />
   <xacro:property name="husky_rear_bumper_extend" value="$(optenv HUSKY_REAR_BUMPER_EXTEND 0)" />
-  <!-- Height of the sensor arch in mm.  Must be either 510 or 300 -->
-  <xacro:arg name="sensor_arch_height"  default="$(optenv HUSKY_SENSOR_ARCH_HEIGHT 510)" />
+  <!-- Height of the sensor arch in mm.  Must be either 540 or 510 or 300 -->
+  <xacro:arg name="sensor_arch_height"  default="$(optenv HUSKY_SENSOR_ARCH_HEIGHT 540)" />
   <xacro:arg name="sensor_arch"         default="$(optenv HUSKY_SENSOR_ARCH 0)" />
+  <xacro:arg name="sensor_arch_xyz"  default="$(optenv HUSKY_SENSOR_ARCH_OFFSET 0.01 0 0)" />
+  <xacro:arg name="sensor_arch_rpy"     default="$(optenv HUSKY_SENSOR_ARCH_RPY 0 0 0)" />
   <xacro:arg name="robot_namespace" default="$(optenv ROBOT_NAMESPACE /)" />
   <xacro:arg name="urdf_extras" default="$(optenv HUSKY_URDF_EXTRAS empty.urdf)" />
@@ -131,6 +133,6 @@
   <link name="imu_link"/>
   <joint name="imu_joint" type="fixed">
-    <origin xyz="$(optenv HUSKY_IMU_XYZ 0.19 0 0.149)" rpy="$(optenv HUSKY_IMU_RPY 0 -1.5708 3.1416)" />
-    <parent link="base_link" />
+    <origin xyz="$(optenv HUSKY_IMU_XYZ 0 0 -0.54)" rpy="$(optenv HUSKY_IMU_RPY 0 -1.5708 3.1416)" />
+    <parent link="sensor_arch_mount_link" />
     <child link="imu_link" />
   </joint>
@@ -140,6 +142,6 @@
   <link name="gps_link"/>
   <joint name="gps_joint" type="fixed">
-    <origin xyz="$(optenv HUSKY_GPS_XYZ 0.0 0.0 0.5)" rpy="$(optenv HUSKY_GPS_RPY 0 0 0)" />
-    <parent link="base_link" />
+    <origin xyz="$(optenv HUSKY_GPS_XYZ -0.1 0 -0.27)" rpy="$(optenv HUSKY_GPS_RPY 0 0 0)" />
+    <parent link="sensor_arch_mount_link" />
     <child link="gps_link" />
   </joint>
@@ -205,6 +207,6 @@
   <xacro:if value="${sensorbar_needed_realsense or sensorbar_needed_zed or sensorbar_user_enabled or sensorbar_needed_lidar or sensorbar_needed_robosense}">
     <xacro:sensor_arch prefix="" parent="top_plate_link" size="$(arg sensor_arch_height)">
-        <origin xyz="$(optenv HUSKY_SENSOR_ARCH_OFFSET 0 0 0)" rpy="$(optenv HUSKY_SENSOR_ARCH_RPY 0 0 0)"/>
-      </xacro:sensor_arch>
+    	<origin xyz="$(arg sensor_arch_xyz)" rpy="$(arg sensor_arch_rpy)"/>
+    </xacro:sensor_arch>
   </xacro:if>
   <!-- add the intel realsense to the sensor arch if needed -->
@@ -228,5 +230,5 @@
       </joint>
       <xacro:zed_camera name="zed_node" model="$(arg zed_model)" parent="zed_mountpoint">
-        <origin xyz="$(arg zed_xyz)" rpy="$(arg zed_rpy)" />
+        <origin xyz="0 0 0" rpy="0 -0.05 0" />
       </xacro:zed_camera>
     </xacro:if>
@@ -245,6 +247,12 @@
   <xacro:unless value="$(arg laser_3d_enabled)">
     <xacro:if value="$(arg robosense_enabled)">
-      <xacro:RS-16 parent="sensor_arch_mount_link" name="robosense" topic="$(optenv HUSKY_ROBOSENSE_TOPIC rs_points)" hz="20" lasers="16" samples="900" collision_range="0.4" min_range="0.4" max_range="150.0" noise="0.008" gpu="true">
-        <origin xyz="$(arg robosense_xyz)" rpy="$(arg robosense_rpy)" />
+	  <joint name="robosense_joint" type="fixed" >
+	    <parent link="sensor_arch_mount_link" />
+		<child link="robosense_mountpoint" />
+		<origin xyz="$(arg robosense_xyz)" rpy="$(arg robosense_rpy)" />
+	  </joint>
+	  <link name="robosense_mountpoint"/>
+      <xacro:RS-16 parent="robosense_mountpoint" name="robosense" topic="$(optenv HUSKY_ROBOSENSE_TOPIC rslidar_points)" hz="20" lasers="16" samples="900" collision_range="0.4" min_range="0.4" max_range="150.0" noise="0.008" gpu="true">
+        <origin xyz="0 0 0.008" rpy="0 0 0" />
       </xacro:RS-16>
     </xacro:if>

Commit message: Tweaking Husky config and parameters

File: husky_description/urdf/husky.urdf.xacro (robot description, xacro)
@@ -44,5 +44,5 @@
   <xacro:arg name="laser_3d_rpy" default="$(optenv HUSKY_LASER_3D_RPY 0 0 0)" />
   <xacro:arg name="robosense_enabled" default="$(optenv HUSKY_ROBOSENSE_ENABLED 1)" />
-  <xacro:arg name="robosense_xyz" default="$(optenv HUSKY_ROBOSENSE_XYZ -0.02 0 0.006)" />
+  <xacro:arg name="robosense_xyz" default="$(optenv HUSKY_ROBOSENSE_XYZ 0 0 0.044)" />
   <xacro:arg name="robosense_rpy" default="$(optenv HUSKY_ROBOSENSE_RPY 0 0 0)" />
   <xacro:arg name="realsense_enabled" default="$(optenv HUSKY_REALSENSE_ENABLED 0)" />
@@ -51,6 +51,6 @@
   <xacro:arg name="realsense_mount" default="$(optenv HUSKY_REALSENSE_MOUNT_FRAME sensor_arch_mount_link)" />
   <xacro:arg name="zed_enabled" default="$(optenv HUSKY_ZED_ENABLED 1)" />
-  <xacro:arg name="zed_xyz" default="$(optenv HUSKY_ZED_XYZ 0 0 -0.025)" />
-  <xacro:arg name="zed_rpy" default="$(optenv HUSKY_ZED_RPY 0 3.141593 0)" />
+  <xacro:arg name="zed_xyz" default="$(optenv HUSKY_ZED_XYZ 0 0 -0.265)" />
+  <xacro:arg name="zed_rpy" default="$(optenv HUSKY_ZED_RPY 0 0.05 0)" />
   <xacro:arg name="zed_mount" default="$(optenv HUSKY_ZED_MOUNT_FRAME sensor_arch_mount_link)" />
   <xacro:arg name="zed_model" default="$(optenv HUSKY_ZED_MODEL zed2)" />
@@ -132,5 +132,5 @@
   <link name="imu_link"/>
   <joint name="imu_joint" type="fixed">
-    <origin xyz="$(optenv HUSKY_IMU_XYZ 0 0 -0.54)" rpy="$(optenv HUSKY_IMU_RPY 0 -1.5708 3.1416)" />
+    <origin xyz="$(optenv HUSKY_IMU_XYZ 0 0 -0.3)" rpy="$(optenv HUSKY_IMU_RPY 3.141593 0 0)" />
     <parent link="sensor_arch_mount_link" />
     <child link="imu_link" />
@@ -141,5 +141,5 @@
   <link name="gps_link"/>
   <joint name="gps_joint" type="fixed">
-    <origin xyz="$(optenv HUSKY_GPS_XYZ -0.1 0 -0.27)" rpy="$(optenv HUSKY_GPS_RPY 0 0 0)" />
+    <origin xyz="$(optenv HUSKY_GPS_XYZ 0 0.22 0)" rpy="$(optenv HUSKY_GPS_RPY 0 0 0)" />
     <parent link="sensor_arch_mount_link" />
     <child link="gps_link" />
@@ -228,6 +228,6 @@
         <child link="zed_mountpoint" />
       </joint>
-      <xacro:zed_camera name="zed_node" model="$(arg zed_model)" parent="zed_mountpoint">
-        <origin xyz="0 0 0" rpy="0 -0.05 0" />
+      <xacro:zed_camera name="zed" model="$(arg zed_model)" parent="zed_mountpoint">
+        <origin xyz="0 0 0" rpy="0 0 0" />
       </xacro:zed_camera>
     </xacro:if>
@@ -246,11 +246,11 @@
   <xacro:unless value="$(arg laser_3d_enabled)">
     <xacro:if value="$(arg robosense_enabled)">
-	  <joint name="robosense_joint" type="fixed" >
-	    <parent link="sensor_arch_mount_link" />
-		<child link="robosense_mountpoint" />
-		<origin xyz="$(arg robosense_xyz)" rpy="$(arg robosense_rpy)" />
-	  </joint>
-	  <link name="robosense_mountpoint"/>
-      <xacro:RS-16 parent="robosense_mountpoint" name="robosense" topic="$(optenv HUSKY_ROBOSENSE_TOPIC rslidar_points)" hz="20" lasers="16" samples="900" collision_range="0.4" min_range="0.4" max_range="150.0" noise="0.008" gpu="true">
+      <joint name="robosense_joint" type="fixed" >
+        <parent link="sensor_arch_mount_link" />
+        <child link="robosense_mountpoint" />
+        <origin xyz="$(arg robosense_xyz)" rpy="$(arg robosense_rpy)" />
+      </joint>
+      <link name="robosense_mountpoint"/>
+      <xacro:RS-16 parent="robosense_mountpoint" name="rslidar" topic="$(optenv HUSKY_ROBOSENSE_TOPIC rslidar_points)" hz="20" lasers="16" samples="900" collision_range="0.4" min_range="0.4" max_range="150.0" noise="0.008" gpu="true">
         <origin xyz="0 0 0.008" rpy="0 0 0" />
       </xacro:RS-16>
@@ -281,5 +281,5 @@
       <robotNamespace>$(arg robot_namespace)</robotNamespace>
       <updateRate>40.0</updateRate>
-      <bodyName>gps_link</bodyName>
+      <bodyName>base_link</bodyName>
       <frameId>gps_link</frameId>
       <topicName>navsat/fix</topicName>

Commit message: Tweaking the kalman filter

File: husky_description/urdf/husky.urdf.xacro (robot description, xacro)
@@ -132,5 +132,5 @@
   <link name="imu_link"/>
   <joint name="imu_joint" type="fixed">
-    <origin xyz="$(optenv HUSKY_IMU_XYZ 0 0 -0.3)" rpy="$(optenv HUSKY_IMU_RPY 3.141593 0 0)" />
+    <origin xyz="$(optenv HUSKY_IMU_XYZ 0 0 -0.3)" rpy="$(optenv HUSKY_IMU_RPY 0 0 0)" />
     <parent link="sensor_arch_mount_link" />
     <child link="imu_link" />
@@ -263,9 +263,10 @@
     </plugin>
   </gazebo>
+  <!--
   <gazebo>
     <plugin name="imu_controller" filename="libhector_gazebo_ros_imu.so">
       <robotNamespace>$(arg robot_namespace)</robotNamespace>
       <updateRate>50.0</updateRate>
-      <bodyName>base_link</bodyName>
+      <bodyName>imu_link</bodyName>
       <topicName>imu/data</topicName>
       <accelDrift>0.005 0.005 0.005</accelDrift>
@@ -277,9 +278,46 @@
     </plugin>
   </gazebo>
+  -->
+  <gazebo reference="imu_link">
+    <gravity>true</gravity>
+    <sensor name="imu_sensor" type="imu">
+      <always_on>true</always_on>
+      <update_rate>100</update_rate>
+      <visualize>true</visualize>
+      <topic>__default_topic__</topic>
+      <plugin filename="libgazebo_ros_imu_sensor.so" name="imu_plugin">
+        <topicName>imu/data</topicName>
+        <bodyName>imu_link</bodyName>
+        <updateRateHZ>50.0</updateRateHZ>
+        <gaussianNoise>0.0</gaussianNoise>
+        <xyzOffset>0 0 0</xyzOffset>
+        <rpyOffset>0 0 0</rpyOffset>
+        <frameName>imu_link</frameName>
+        <initialOrientationAsReference>false</initialOrientationAsReference>
+      </plugin>
+      <pose>0 0 0 0 0 0</pose>
+    </sensor>
+  </gazebo>
+  <gazebo reference="imu_link">
+    <plugin name="magnetometer_controller" filename="libhector_gazebo_ros_magnetic.so">
+      <alwaysOn>true</alwaysOn>
+      <updateRate>50.0</updateRate>
+      <bodyName>imu_link</bodyName>
+      <topicName>imu/mag</topicName>
+      <offset>0 0 0</offset>
+      <drift>0.0 0.0 0.0</drift>
+      <gaussianNoise>0.0 0.0 0.0</gaussianNoise>
+      <declination>1.433</declination>
+      <inclination>64.233</inclination>
+      <magnitude>0.0000482567</magnitude>
+      <referenceHeading>0</referenceHeading>
+      <useMagneticFieldMsgs>true</useMagneticFieldMsgs>
+    </plugin>
+  </gazebo>
   <gazebo>
     <plugin name="gps_controller" filename="libhector_gazebo_ros_gps.so">
       <robotNamespace>$(arg robot_namespace)</robotNamespace>
-      <updateRate>40.0</updateRate>
-      <bodyName>base_link</bodyName>
+      <updateRate>10.0</updateRate>
+      <bodyName>gps_link</bodyName>
       <frameId>gps_link</frameId>
       <topicName>navsat/fix</topicName>

Commit message: Tweaking the kalman filter

File: husky_description/urdf/husky.urdf.xacro (robot description, xacro)
@@ -133,5 +133,5 @@
   <link name="imu_link"/>
   <joint name="imu_joint" type="fixed">
-    <origin xyz="$(optenv HUSKY_IMU_XYZ 0 0 -0.3)" rpy="$(optenv HUSKY_IMU_RPY 3.141593 0 0)" />
+    <origin xyz="$(optenv HUSKY_IMU_XYZ 0 0 -0.3)" rpy="$(optenv HUSKY_IMU_RPY 0 0 0)" />
     <parent link="sensor_arch_mount_link" />
     <child link="imu_link" />
@@ -264,9 +264,10 @@
     </plugin>
   </gazebo>
+  <!--
   <gazebo>
     <plugin name="imu_controller" filename="libhector_gazebo_ros_imu.so">
       <robotNamespace>$(arg robot_namespace)</robotNamespace>
       <updateRate>50.0</updateRate>
-      <bodyName>base_link</bodyName>
+      <bodyName>imu_link</bodyName>
       <topicName>imu/data</topicName>
       <accelDrift>0.005 0.005 0.005</accelDrift>
@@ -278,9 +279,46 @@
     </plugin>
   </gazebo>
+  -->
+  <gazebo reference="imu_link">
+    <gravity>true</gravity>
+    <sensor name="imu_sensor" type="imu">
+      <always_on>true</always_on>
+      <update_rate>100</update_rate>
+      <visualize>true</visualize>
+      <topic>__default_topic__</topic>
+      <plugin filename="libgazebo_ros_imu_sensor.so" name="imu_plugin">
+        <topicName>imu/data</topicName>
+        <bodyName>imu_link</bodyName>
+        <updateRateHZ>50.0</updateRateHZ>
+        <gaussianNoise>0.0</gaussianNoise>
+        <xyzOffset>0 0 0</xyzOffset>
+        <rpyOffset>0 0 0</rpyOffset>
+        <frameName>imu_link</frameName>
+        <initialOrientationAsReference>false</initialOrientationAsReference>
+      </plugin>
+      <pose>0 0 0 0 0 0</pose>
+    </sensor>
+  </gazebo>
+  <gazebo reference="imu_link">
+    <plugin name="magnetometer_controller" filename="libhector_gazebo_ros_magnetic.so">
+      <alwaysOn>true</alwaysOn>
+      <updateRate>50.0</updateRate>
+      <bodyName>imu_link</bodyName>
+      <topicName>imu/mag</topicName>
+      <offset>0 0 0</offset>
+      <drift>0.0 0.0 0.0</drift>
+      <gaussianNoise>0.0 0.0 0.0</gaussianNoise>
+      <declination>1.433</declination>
+      <inclination>64.233</inclination>
+      <magnitude>0.0000482567</magnitude>
+      <referenceHeading>0</referenceHeading>
+      <useMagneticFieldMsgs>true</useMagneticFieldMsgs>
+    </plugin>
+  </gazebo>
   <gazebo>
     <plugin name="gps_controller" filename="libhector_gazebo_ros_gps.so">
       <robotNamespace>$(arg robot_namespace)</robotNamespace>
-      <updateRate>40.0</updateRate>
-      <bodyName>base_link</bodyName>
+      <updateRate>10.0</updateRate>
+      <bodyName>gps_link</bodyName>
       <frameId>gps_link</frameId>
       <topicName>navsat/fix</topicName>

Commit message: Tweaking heading parameters.. again

File: husky_description/urdf/husky.urdf.xacro (robot description, xacro)
@@ -22,4 +22,5 @@
 -->
 <robot name="husky" xmlns:xacro="http://ros.org/wiki/xacro">
+  <xacro:arg name="husky_sim" default="$(optenv HUSKY_SIM 0)" />
   <xacro:arg name="laser_enabled" default="$(optenv HUSKY_LMS1XX_ENABLED 0)" />
   <xacro:arg name="laser_xyz" default="$(optenv HUSKY_LMS1XX_XYZ 0.2206 0.0 0.00635)" />
@@ -132,9 +133,18 @@
   <!-- Can be modified with environment variables in /etc/ros/setup.bash -->
   <link name="imu_link"/>
-  <joint name="imu_joint" type="fixed">
-    <origin xyz="$(optenv HUSKY_IMU_XYZ 0 0 -0.3)" rpy="$(optenv HUSKY_IMU_RPY 0 0 0)" />
-    <parent link="sensor_arch_mount_link" />
-    <child link="imu_link" />
-  </joint>
+  <xacro:if value="$(arg husky_sim)">
+    <joint name="imu_joint" type="fixed">
+      <origin xyz="$(optenv HUSKY_IMU_XYZ 0 0 -0.3)" rpy="$(optenv HUSKY_IMU_RPY 0 3.141593 3.141593)" />
+      <parent link="sensor_arch_mount_link" />
+      <child link="imu_link" />
+    </joint>
+  </xacro:if>
+  <xacro:unless value="$(arg husky_sim)">
+    <joint name="imu_joint" type="fixed">
+      <origin xyz="$(optenv HUSKY_IMU_XYZ 0 0 -0.3)" rpy="$(optenv HUSKY_IMU_RPY 0 3.141593 3.141593)" />
+      <parent link="sensor_arch_mount_link" />
+      <child link="imu_link" />
+    </joint>
+  </xacro:unless>
   <gazebo reference="imu_link">
   </gazebo>

Commit message: Tweaking heading parameters.. again

File: husky_description/urdf/husky.urdf.xacro (robot description, xacro)
@@ -22,4 +22,5 @@
 -->
 <robot name="husky" xmlns:xacro="http://ros.org/wiki/xacro">
+  <xacro:arg name="husky_sim" default="$(optenv HUSKY_SIM 0)" />
   <xacro:arg name="laser_enabled" default="$(optenv HUSKY_LMS1XX_ENABLED 0)" />
   <xacro:arg name="laser_xyz" default="$(optenv HUSKY_LMS1XX_XYZ 0.2206 0.0 0.00635)" />
@@ -131,9 +132,18 @@
   <!-- Can be modified with environment variables in /etc/ros/setup.bash -->
   <link name="imu_link"/>
-  <joint name="imu_joint" type="fixed">
-    <origin xyz="$(optenv HUSKY_IMU_XYZ 0 0 -0.3)" rpy="$(optenv HUSKY_IMU_RPY 0 0 0)" />
-    <parent link="sensor_arch_mount_link" />
-    <child link="imu_link" />
-  </joint>
+  <xacro:if value="$(arg husky_sim)">
+    <joint name="imu_joint" type="fixed">
+      <origin xyz="$(optenv HUSKY_IMU_XYZ 0 0 -0.3)" rpy="$(optenv HUSKY_IMU_RPY 0 3.141593 3.141593)" />
+      <parent link="sensor_arch_mount_link" />
+      <child link="imu_link" />
+    </joint>
+  </xacro:if>
+  <xacro:unless value="$(arg husky_sim)">
+    <joint name="imu_joint" type="fixed">
+      <origin xyz="$(optenv HUSKY_IMU_XYZ 0 0 -0.3)" rpy="$(optenv HUSKY_IMU_RPY 0 3.141593 3.141593)" />
+      <parent link="sensor_arch_mount_link" />
+      <child link="imu_link" />
+    </joint>
+  </xacro:unless>
   <gazebo reference="imu_link">
   </gazebo>
