Commit message: Post CoHoMa version with customizable config in husky_bringup, new lidar robosense driver (robosense_sdk)

File: husky_description/urdf/husky.urdf.xacro (robot description, xacro)
@@ -45,5 +45,5 @@
   <xacro:arg name="laser_3d_rpy" default="$(optenv HUSKY_LASER_3D_RPY 0 0 0)" />
   <xacro:arg name="robosense_enabled" default="$(optenv HUSKY_ROBOSENSE_ENABLED 1)" />
-  <xacro:arg name="robosense_xyz" default="$(optenv HUSKY_ROBOSENSE_XYZ 0 0 0.044)" />
+  <xacro:arg name="robosense_xyz" default="$(optenv HUSKY_ROBOSENSE_XYZ 0.017 0 -0.135)" />
   <xacro:arg name="robosense_rpy" default="$(optenv HUSKY_ROBOSENSE_RPY 0 0 0)" />
   <xacro:arg name="realsense_enabled" default="$(optenv HUSKY_REALSENSE_ENABLED 0)" />
@@ -70,10 +70,14 @@
   <xacro:include filename="$(find husky_description)/urdf/wheel.urdf.xacro" />
   <xacro:include filename="$(find husky_description)/urdf/accessories/intel_realsense.urdf.xacro"/>
-  <xacro:include filename="$(find husky_description)/urdf/accessories/zed_macro.urdf.xacro" />
+  <xacro:if value="$(arg zed_enabled)">
+    <xacro:include filename="$(find husky_description)/urdf/accessories/zed_macro.urdf.xacro" />
+  </xacro:if>
   <xacro:include filename="$(find husky_description)/urdf/accessories/hokuyo_ust10.urdf.xacro" />
   <xacro:include filename="$(find husky_description)/urdf/accessories/sick_lms1xx_mount.urdf.xacro"/>
   <xacro:include filename="$(find husky_description)/urdf/accessories/sensor_arch.urdf.xacro"/>
   <xacro:include filename="$(find husky_description)/urdf/accessories/vlp16_mount.urdf.xacro"/>
-  <xacro:include filename="$(find husky_description)/urdf/accessories/RS-16.urdf.xacro"/>
+  <xacro:if value="$(arg robosense_enabled)">
+    <xacro:include filename="$(find husky_description)/urdf/accessories/RS-16.urdf.xacro"/>
+  </xacro:if>
   <xacro:property name="M_PI" value="3.14159"/>
   <!-- Base Size -->
@@ -134,5 +138,5 @@
   <xacro:if value="$(arg husky_sim)">
     <joint name="imu_joint" type="fixed">
-      <origin xyz="$(optenv HUSKY_IMU_XYZ 0 0 -0.3)" rpy="$(optenv HUSKY_IMU_RPY 0 3.141593 3.141593)" />
+      <origin xyz="$(optenv HUSKY_IMU_XYZ 0 0 -0.3)" rpy="$(optenv HUSKY_IMU_RPY 0 -1.5708 3.1416)" />
       <parent link="sensor_arch_mount_link" />
       <child link="imu_link" />
@@ -141,5 +145,5 @@
   <xacro:unless value="$(arg husky_sim)">
     <joint name="imu_joint" type="fixed">
-      <origin xyz="$(optenv HUSKY_IMU_XYZ 0 0 -0.3)" rpy="$(optenv HUSKY_IMU_RPY 0 3.141593 3.141593)" />
+      <origin xyz="$(optenv HUSKY_IMU_XYZ 0 0 -0.3)" rpy="$(optenv HUSKY_IMU_RPY 0 0 0)" />
       <parent link="sensor_arch_mount_link" />
       <child link="imu_link" />

Commit message: Post CoHoMa version with customizable config in husky_bringup, new lidar robosense driver (robosense_sdk)

File: husky_description/urdf/husky.urdf.xacro (robot description, xacro)
@@ -45,5 +45,5 @@
   <xacro:arg name="laser_3d_rpy" default="$(optenv HUSKY_LASER_3D_RPY 0 0 0)" />
   <xacro:arg name="robosense_enabled" default="$(optenv HUSKY_ROBOSENSE_ENABLED 1)" />
-  <xacro:arg name="robosense_xyz" default="$(optenv HUSKY_ROBOSENSE_XYZ 0 0 0.044)" />
+  <xacro:arg name="robosense_xyz" default="$(optenv HUSKY_ROBOSENSE_XYZ 0.017 0 -0.135)" />
   <xacro:arg name="robosense_rpy" default="$(optenv HUSKY_ROBOSENSE_RPY 0 0 0)" />
   <xacro:arg name="realsense_enabled" default="$(optenv HUSKY_REALSENSE_ENABLED 0)" />
@@ -70,5 +70,7 @@
   <xacro:include filename="$(find husky_description)/urdf/wheel.urdf.xacro" />
   <xacro:include filename="$(find husky_description)/urdf/accessories/intel_realsense.urdf.xacro"/>
-  <xacro:include filename="$(find husky_description)/urdf/accessories/zed_macro.urdf.xacro" />
+  <xacro:if value="$(arg zed_enabled)">
+    <xacro:include filename="$(find husky_description)/urdf/accessories/zed_macro.urdf.xacro" />
+  </xacro:if>
   <xacro:include filename="$(find husky_description)/urdf/accessories/hokuyo_ust10.urdf.xacro" />
   <xacro:include filename="$(find husky_description)/urdf/accessories/sick_lms1xx_mount.urdf.xacro"/>
@@ -76,5 +78,7 @@
   <xacro:include filename="$(find husky_description)/urdf/accessories/hokuyo_ust10.urdf.xacro"/>
   <xacro:include filename="$(find husky_description)/urdf/accessories/vlp16_mount.urdf.xacro"/>
-  <xacro:include filename="$(find husky_description)/urdf/accessories/RS-16.urdf.xacro"/>
+  <xacro:if value="$(arg robosense_enabled)">
+    <xacro:include filename="$(find husky_description)/urdf/accessories/RS-16.urdf.xacro"/>
+  </xacro:if>
   <xacro:property name="M_PI" value="3.14159"/>
   <!-- Base Size -->
@@ -135,5 +139,5 @@
   <xacro:if value="$(arg husky_sim)">
     <joint name="imu_joint" type="fixed">
-      <origin xyz="$(optenv HUSKY_IMU_XYZ 0 0 -0.3)" rpy="$(optenv HUSKY_IMU_RPY 0 3.141593 3.141593)" />
+      <origin xyz="$(optenv HUSKY_IMU_XYZ 0 0 -0.3)" rpy="$(optenv HUSKY_IMU_RPY 0 -1.5708 3.1416)" />
       <parent link="sensor_arch_mount_link" />
       <child link="imu_link" />
@@ -142,5 +146,5 @@
   <xacro:unless value="$(arg husky_sim)">
     <joint name="imu_joint" type="fixed">
-      <origin xyz="$(optenv HUSKY_IMU_XYZ 0 0 -0.3)" rpy="$(optenv HUSKY_IMU_RPY 0 3.141593 3.141593)" />
+      <origin xyz="$(optenv HUSKY_IMU_XYZ 0 0 -0.3)" rpy="$(optenv HUSKY_IMU_RPY 0 0 0)" />
       <parent link="sensor_arch_mount_link" />
       <child link="imu_link" />

Commit message: Setting new architecture description, modifying localization configuration because of SBG IMU drivers (/imu/data message) has been changed to point toward 0 when facing East, actually adding web_video_server and possibility to record rosbag on external disk

File: husky_description/urdf/husky.urdf.xacro (robot description, xacro)
@@ -45,5 +45,5 @@
   <xacro:arg name="laser_3d_rpy" default="$(optenv HUSKY_LASER_3D_RPY 0 0 0)" />
   <xacro:arg name="robosense_enabled" default="$(optenv HUSKY_ROBOSENSE_ENABLED 1)" />
-  <xacro:arg name="robosense_xyz" default="$(optenv HUSKY_ROBOSENSE_XYZ 0.017 0 -0.135)" />
+  <xacro:arg name="robosense_xyz" default="$(optenv HUSKY_ROBOSENSE_XYZ 0 0 -0.33)" />
   <xacro:arg name="robosense_rpy" default="$(optenv HUSKY_ROBOSENSE_RPY 0 0 0)" />
   <xacro:arg name="realsense_enabled" default="$(optenv HUSKY_REALSENSE_ENABLED 0)" />
@@ -52,12 +52,12 @@
   <xacro:arg name="realsense_mount" default="$(optenv HUSKY_REALSENSE_MOUNT_FRAME sensor_arch_mount_link)" />
   <xacro:arg name="zed_enabled" default="$(optenv HUSKY_ZED_ENABLED 1)" />
-  <xacro:arg name="zed_xyz" default="$(optenv HUSKY_ZED_XYZ 0 0 -0.265)" />
-  <xacro:arg name="zed_rpy" default="$(optenv HUSKY_ZED_RPY 0 0.05 0)" />
+  <xacro:arg name="zed_xyz" default="$(optenv HUSKY_ZED_XYZ 0 0 -0.18)" />
+  <xacro:arg name="zed_rpy" default="$(optenv HUSKY_ZED_RPY 0 0.197 0)" />
   <xacro:arg name="zed_mount" default="$(optenv HUSKY_ZED_MOUNT_FRAME sensor_arch_mount_link)" />
   <xacro:arg name="zed_model" default="$(optenv HUSKY_ZED_MODEL zed2)" />
   <xacro:property name="husky_front_bumper_extend" value="$(optenv HUSKY_FRONT_BUMPER_EXTEND 0)" />
   <xacro:property name="husky_rear_bumper_extend" value="$(optenv HUSKY_REAR_BUMPER_EXTEND 0)" />
-  <!-- Height of the sensor arch in mm.  Must be either 540 or 510 or 300 -->
-  <xacro:arg name="sensor_arch_height"  default="$(optenv HUSKY_SENSOR_ARCH_HEIGHT 540)" />
+  <!-- Height of the sensor arch in mm.  Must be either 560 or 540 or 510 or 300 -->
+  <xacro:arg name="sensor_arch_height"  default="$(optenv HUSKY_SENSOR_ARCH_HEIGHT 560)" />
   <xacro:arg name="sensor_arch"         default="$(optenv HUSKY_SENSOR_ARCH 0)" />
   <xacro:arg name="sensor_arch_xyz"  default="$(optenv HUSKY_SENSOR_ARCH_OFFSET 0.01 0 0)" />
@@ -138,5 +138,5 @@
   <xacro:if value="$(arg husky_sim)">
     <joint name="imu_joint" type="fixed">
-      <origin xyz="$(optenv HUSKY_IMU_XYZ 0 0 -0.3)" rpy="$(optenv HUSKY_IMU_RPY 0 -1.5708 3.1416)" />
+      <origin xyz="$(optenv HUSKY_IMU_XYZ 0 0 -0.38)" rpy="$(optenv HUSKY_IMU_RPY 0 0 0)" />
       <parent link="sensor_arch_mount_link" />
       <child link="imu_link" />
@@ -145,5 +145,5 @@
   <xacro:unless value="$(arg husky_sim)">
     <joint name="imu_joint" type="fixed">
-      <origin xyz="$(optenv HUSKY_IMU_XYZ 0 0 -0.3)" rpy="$(optenv HUSKY_IMU_RPY 0 0 0)" />
+      <origin xyz="$(optenv HUSKY_IMU_XYZ 0 0 -0.38)" rpy="$(optenv HUSKY_IMU_RPY 0 0 0)" />
       <parent link="sensor_arch_mount_link" />
       <child link="imu_link" />
@@ -152,8 +152,21 @@
   <gazebo reference="imu_link">
   </gazebo>
+  <!-- GNSS Links is the standard mounting position for the SBG IMU dual GNSS-->
+  <link name="left_imu_gnss_link"/>
+  <joint name="left_imu_gnss_joint" type="fixed">
+    <origin xyz="0 0.25 0.01" rpy="0 0 0" />
+    <parent link="sensor_arch_mount_link" />
+    <child link="left_imu_gnss_link" />
+  </joint>
+  <link name="right_imu_gnss_link"/>
+  <joint name="right_imu_gnss_joint" type="fixed">
+    <origin xyz="0 -0.25 0.01" rpy="0 0 0" />
+    <parent link="sensor_arch_mount_link" />
+    <child link="right_imu_gnss_link" />
+  </joint>
   <!-- GPS Link is the standard mounting position for the GPS-->
   <link name="gps_link"/>
   <joint name="gps_joint" type="fixed">
-    <origin xyz="$(optenv HUSKY_GPS_XYZ 0 0.22 0)" rpy="$(optenv HUSKY_GPS_RPY 0 0 0)" />
+    <origin xyz="$(optenv HUSKY_GPS_XYZ 0 0.2 0.01)" rpy="$(optenv HUSKY_GPS_RPY 0 0 0)" />
     <parent link="sensor_arch_mount_link" />
     <child link="gps_link" />
